Commit message: fixed position of  mounting link, now it's flush with the mounting holes.
The ft300_mounting_plate link was not flush with the mounting holes. Therefore, connecting the link directly to an UR robot would previously have resulted in an offset.

File: robotiq_ft_sensor_description/urdf/robotiq_ft300.urdf.xacro (robot description, xacro)
@@ -34,5 +34,5 @@
         <link name="${tf_prefix}ft300_mounting_plate">
             <visual>
-                <origin xyz="0 0 0" rpy="0 0 0" />
+                <origin xyz="0 0 -0.004" rpy="0 0 0" />
                 <geometry>
                     <mesh filename="file://$(find robotiq_ft_sensor_description)/meshes/visual/mountings/robotiq_ft300-G-062-COUPLING_G-50-4M6-1D6_20181119.STL"/>
@@ -43,5 +43,5 @@
             </visual>
             <collision>
-                <origin xyz="0 0 0" rpy="0 0 0" />
+                <origin xyz="0 0 0" rpy="0 0 -0.004" />
                 <geometry>
                     <mesh filename="file://$(find robotiq_ft_sensor_description)/meshes/collision/mountings/robotiq_ft300-G-062-COUPLING_G-50-4M6-1D6_20181119.STL"/>
@@ -51,5 +51,5 @@
          <!-- Connect force sensor with mounting/coupling plate -->
         <joint name="${tf_prefix}ft300_mounting_plate_joint" type="fixed">
-            <origin xyz="0 0 0.0415" rpy="0 ${pi} 0"/>
+            <origin xyz="0 0 0.0375" rpy="0 ${pi} 0"/>
             <parent link="${tf_prefix}ft300_mounting_plate" />
             <child link="${tf_prefix}ft300_sensor" />
